Commit message: Kinova

File: kinova/src/kinova-ros/kinova_description/urdf/j2s6s300.xacro (robot description, xacro)
@@ -1,19 +1,9 @@
 <?xml version="1.0"?>
 <!-- j2_6s refers to jaco v2 6DOF spherical -->
-<robot xmlns:xi="http://www.w3.org/2001/XInclude"
-    xmlns:gazebo="http://playerstage.sourceforge.net/gazebo/xmlschema/#gz"
-    xmlns:model="http://playerstage.sourceforge.net/gazebo/xmlschema/#model"
-    xmlns:sensor="http://playerstage.sourceforge.net/gazebo/xmlschema/#sensor"
-    xmlns:body="http://playerstage.sourceforge.net/gazebo/xmlschema/#body"
-    xmlns:geom="http://playerstage.sourceforge.net/gazebo/xmlschema/#geom"
-    xmlns:joint="http://playerstage.sourceforge.net/gazebo/xmlschema/#joint"
-    xmlns:controller="http://playerstage.sourceforge.net/gazebo/xmlschema/#controller"
-    xmlns:interface="http://playerstage.sourceforge.net/gazebo/xmlschema/#interface"
-    xmlns:rendering="http://playerstage.sourceforge.net/gazebo/xmlschema/#rendering"
-    xmlns:renderable="http://playerstage.sourceforge.net/gazebo/xmlschema/#renderable"
-    xmlns:physics="http://playerstage.sourceforge.net/gazebo/xmlschema/#physics"
-    xmlns:xacro="http://www.ros.org/wiki/xacro">
+<robot name="j2s6s300" xmlns:xacro="http://www.ros.org/wiki/xacro">
+    <xacro:property name="M_PI" value="3.14159274"/>
     <xacro:include filename="$(find kinova_description)/urdf/kinova_common.xacro" />
     <xacro:include filename="$(find kinova_description)/urdf/kinova_finger_set.xacro" />
+    <xacro:include filename="$(find kinova_description)/urdf/camera/camera.urdf.xacro"/>
     <!-- Import all Gazebo-customization elements -->
     <xacro:include filename="$(find kinova_description)/urdf/kinova.gazebo" />
@@ -51,5 +41,5 @@
     <xacro:property name="joint_1_upper_limit" value="${2*J_PI}" />
     <xacro:property name="joint_1_velocity_limit" value="${36*J_PI/180}" />
-    <xacro:property name="joint_1_torque_limit" value="40" />
+    <xacro:property name="joint_1_torque_limit" value="120" />
     <xacro:property name="joint_2" value="joint_2" />
     <xacro:property name="joint_2_type" value="revolute" />
@@ -60,5 +50,5 @@
     <xacro:property name="joint_2_upper_limit" value="${313/180*J_PI}" />
     <xacro:property name="joint_2_velocity_limit" value="${36*J_PI/180}" />
-    <xacro:property name="joint_2_torque_limit" value="80" />
+    <xacro:property name="joint_2_torque_limit" value="240" />
     <xacro:property name="joint_3" value="joint_3" />
     <xacro:property name="joint_3_type" value="revolute" />
@@ -69,5 +59,5 @@
     <xacro:property name="joint_3_upper_limit" value="${341/180*J_PI}" />
     <xacro:property name="joint_3_velocity_limit" value="${36*J_PI/180}" />
-    <xacro:property name="joint_3_torque_limit" value="40" />
+    <xacro:property name="joint_3_torque_limit" value="120" />
     <xacro:property name="joint_4" value="joint_4" />
     <xacro:property name="joint_4_type" value="continuous" />
@@ -78,5 +68,5 @@
     <xacro:property name="joint_4_upper_limit" value="${2*J_PI}" />
     <xacro:property name="joint_4_velocity_limit" value="${48*J_PI/180}" />
-    <xacro:property name="joint_4_torque_limit" value="20" />
+    <xacro:property name="joint_4_torque_limit" value="60" />
     <xacro:property name="joint_5" value="joint_5" />
     <xacro:property name="joint_5_type" value="revolute" />
@@ -87,5 +77,5 @@
     <xacro:property name="joint_5_upper_limit" value="${330/180*J_PI}" />
     <xacro:property name="joint_5_velocity_limit" value="${48*J_PI/180}" />
-    <xacro:property name="joint_5_torque_limit" value="20" />
+    <xacro:property name="joint_5_torque_limit" value="60" />
     <xacro:property name="joint_6" value="joint_6" />
     <xacro:property name="joint_6_type" value="continuous" />
@@ -96,5 +86,5 @@
     <xacro:property name="joint_6_upper_limit" value="${2*J_PI}" />
     <xacro:property name="joint_6_velocity_limit" value="${48*J_PI/180}" />
-    <xacro:property name="joint_6_torque_limit" value="20" />
+    <xacro:property name="joint_6_torque_limit" value="60" />
     <xacro:property name="joint_end_effector" value="end_effector_offset" />
     <xacro:property name="joint_end_effector_type" value="fixed" />
@@ -106,4 +96,8 @@
         <xacro:kinova_armlink link_name="${prefix}_link_base" link_mesh="${link_base_mesh}" mesh_no="${link_base_mesh_no}"/>
         <xacro:kinova_armjoint joint_name="${prefix}_joint_base" type="${joint_base_type}" parent="${base_parent}" child="${prefix}_link_base" joint_axis_xyz="${joint_base_axis_xyz}" joint_origin_xyz="${joint_base_origin_xyz}" joint_origin_rpy="${joint_base_origin_rpy}" joint_lower_limit="0" joint_upper_limit="0" joint_velocity_limit="0" joint_torque_limit="0" fixed="true"/>
+       <!-- Camera -->
+       <xacro:camera_v0 parent="${prefix}_link_base">
+	     <origin xyz="0.4 0.4 0.5" rpy="0 ${M_PI/4} ${-M_PI/2}"/>
+       </xacro:camera_v0>
         <xacro:kinova_armlink link_name="${prefix}_link_1" link_mesh="${link_1_mesh}" use_ring_mesh="true" mesh_no="${link_1_mesh_no}"/>
         <xacro:kinova_armjoint joint_name="${prefix}_joint_1" type="${joint_1_type}" parent="${prefix}_link_base" child="${prefix}_link_1" joint_axis_xyz="${joint_1_axis_xyz}" joint_origin_xyz="${joint_1_origin_xyz}" joint_origin_rpy="${joint_1_origin_rpy}" joint_lower_limit="${joint_1_lower_limit}" joint_upper_limit="${joint_1_upper_limit}" joint_velocity_limit="${joint_1_velocity_limit}" joint_torque_limit="${joint_1_torque_limit}"/>
@@ -122,3 +116,5 @@
     <xacro:kinova_3fingers link_hand="${prefix}_link_6" prefix="${prefix}_"/>
     </xacro:macro>
+    <!-- camera -->
+    <xacro:camera_gazebo_v0 />
 </robot>

File: kinova/src/kinova-ros/kinova_description/urdf/j2s6s300_standalone.xacro (robot description, xacro)
@@ -2,16 +2,16 @@
 <!-- j2s6_3 refers to jaco v2 6DOF spherical 3fingers -->
 <robot xmlns:xi="http://www.w3.org/2001/XInclude"
-	xmlns:gazebo="http://playerstage.sourceforge.net/gazebo/xmlschema/#gz"
-    xmlns:model="http://playerstage.sourceforge.net/gazebo/xmlschema/#model"
-	xmlns:sensor="http://playerstage.sourceforge.net/gazebo/xmlschema/#sensor"
-	xmlns:body="http://playerstage.sourceforge.net/gazebo/xmlschema/#body"
-    xmlns:geom="http://playerstage.sourceforge.net/gazebo/xmlschema/#geom"
-    xmlns:joint="http://playerstage.sourceforge.net/gazebo/xmlschema/#joint"
-	xmlns:controller="http://playerstage.sourceforge.net/gazebo/xmlschema/#controller"
-	xmlns:interface="http://playerstage.sourceforge.net/gazebo/xmlschema/#interface"
-	xmlns:rendering="http://playerstage.sourceforge.net/gazebo/xmlschema/#rendering"
-    xmlns:renderable="http://playerstage.sourceforge.net/gazebo/xmlschema/#renderable"
-    xmlns:physics="http://playerstage.sourceforge.net/gazebo/xmlschema/#physics"
-	xmlns:xacro="http://www.ros.org/wiki/xacro" name="j2s6s300">
+       xmlns:gazebo="http://playerstage.sourceforge.net/gazebo/xmlschema/#gz"
+       xmlns:model="http://playerstage.sourceforge.net/gazebo/xmlschema/#model"
+       xmlns:sensor="http://playerstage.sourceforge.net/gazebo/xmlschema/#sensor"
+       xmlns:body="http://playerstage.sourceforge.net/gazebo/xmlschema/#body"
+       xmlns:geom="http://playerstage.sourceforge.net/gazebo/xmlschema/#geom"
+       xmlns:joint="http://playerstage.sourceforge.net/gazebo/xmlschema/#joint"
+       xmlns:controller="http://playerstage.sourceforge.net/gazebo/xmlschema/#controller"
+       xmlns:interface="http://playerstage.sourceforge.net/gazebo/xmlschema/#interface"
+       xmlns:rendering="http://playerstage.sourceforge.net/gazebo/xmlschema/#rendering"
+       xmlns:renderable="http://playerstage.sourceforge.net/gazebo/xmlschema/#renderable"
+       xmlns:physics="http://playerstage.sourceforge.net/gazebo/xmlschema/#physics"
+       xmlns:xacro="http://www.ros.org/wiki/xacro" name="j2s6s300">
   <xacro:include filename="$(find kinova_description)/urdf/j2s6s300.xacro"/>
   <link name="root"/>

File: kinova/src/kinova-ros/kinova_description/urdf/kinova_common.xacro (robot description, xacro)
@@ -99,4 +99,5 @@
      </transmission>
      <!--For torque sensing in simulation-->
+     <!--
      <gazebo reference="${joint_name}">
         <provideFeedback>true</provideFeedback>
@@ -109,4 +110,5 @@
         </plugin>
       </gazebo>
+      -->
      </xacro:unless>
   </xacro:macro>
@@ -132,5 +134,5 @@
             <axis xyz="0 0 1"/>
             <origin xyz="${finger_origin_xyz}" rpy="${finger_origin_rpy}"/>
-            <limit lower="0" upper="1.51" effort="2" velocity="1"/>
+            <limit lower="0" upper="1.51" effort="10" velocity="1"/>
         </joint>
 		    <transmission name="${prefix}joint_finger_${finger_number}_trans">
@@ -150,5 +152,5 @@
             <axis xyz="0 0 1"/>
             <origin xyz="0.044 -0.003 0" rpy="0 0 0"/>
-            <limit lower="0" upper="2" effort="2" velocity="1"/>
+            <limit lower="0" upper="2" effort="10" velocity="1"/>
         </joint>
         <transmission name="${prefix}joint_finger_tip_${finger_number}_trans">
