Commit message: MoveIT para el Mico (no funciona)

File: kinova_roscontrol/src/kinova-ros/kinova_moveit_mico/config/gazebo_m1n6s300.urdf (robot description, URDF)
Before this commit: robot j2n6s300, 17 links, 16 joints
Links:
- removed link j2n6s300_end_effector
- removed link j2n6s300_link_1
- removed link j2n6s300_link_2
- removed link j2n6s300_link_3
- removed link j2n6s300_link_4
- removed link j2n6s300_link_5
- removed link j2n6s300_link_6
- removed link j2n6s300_link_base
- removed link j2n6s300_link_finger_1
- removed link j2n6s300_link_finger_2
- removed link j2n6s300_link_finger_3
- removed link j2n6s300_link_finger_tip_1
- removed link j2n6s300_link_finger_tip_2
- removed link j2n6s300_link_finger_tip_3
- added link m1n6s300_end_effector
- added link m1n6s300_link_1, mass 0.7477; collision mesh filename=package://kinova_description/meshes/shoulder.dae; visual mesh filename=package://kinova_description/meshes/ring_big.dae
- added link m1n6s300_link_2, mass 0.85968; collision mesh filename=package://kinova_description/meshes/arm_mico.dae; visual mesh filename=package://kinova_description/meshes/arm_mico.dae
- added link m1n6s300_link_3, mass 0.606; collision mesh filename=package://kinova_description/meshes/forearm_mico.dae; visual mesh filename=package://kinova_description/meshes/forearm_mico.dae
- added link m1n6s300_link_4, mass 0.426367; collision mesh filename=package://kinova_description/meshes/wrist.dae; visual mesh filename=package://kinova_description/meshes/ring_small.dae
- added link m1n6s300_link_5, mass 0.426367; collision mesh filename=package://kinova_description/meshes/wrist.dae; visual mesh filename=package://kinova_description/meshes/ring_small.dae
- added link m1n6s300_link_6, mass 0.99; collision mesh filename=package://kinova_description/meshes/hand_3finger.dae; visual mesh filename=package://kinova_description/meshes/hand_3finger.dae
- added link m1n6s300_link_base, mass 0.46784; collision mesh filename=package://kinova_description/meshes/base.dae; visual mesh filename=package://kinova_description/meshes/base.dae
- added link m1n6s300_link_finger_1, mass 0.01; collision mesh filename=package://kinova_description/meshes/finger_proximal.dae; visual mesh filename=package://kinova_description/meshes/finger_proximal.dae
- added link m1n6s300_link_finger_2, mass 0.01; collision mesh filename=package://kinova_description/meshes/finger_proximal.dae; visual mesh filename=package://kinova_description/meshes/finger_proximal.dae
- added link m1n6s300_link_finger_3, mass 0.01; collision mesh filename=package://kinova_description/meshes/finger_proximal.dae; visual mesh filename=package://kinova_description/meshes/finger_proximal.dae
- added link m1n6s300_link_finger_tip_1, mass 0.01; collision mesh filename=package://kinova_description/meshes/finger_distal.dae; visual mesh filename=package://kinova_description/meshes/finger_distal.dae
- added link m1n6s300_link_finger_tip_2, mass 0.01; collision mesh filename=package://kinova_description/meshes/finger_distal.dae; visual mesh filename=package://kinova_description/meshes/finger_distal.dae
- added link m1n6s300_link_finger_tip_3, mass 0.01; collision mesh filename=package://kinova_description/meshes/finger_distal.dae; visual mesh filename=package://kinova_description/meshes/finger_distal.dae
Joints:
- removed joint j2n6s300_joint_1
- removed joint j2n6s300_joint_2
- removed joint j2n6s300_joint_3
- removed joint j2n6s300_joint_4
- removed joint j2n6s300_joint_5
- removed joint j2n6s300_joint_6
- removed joint j2n6s300_joint_base
- removed joint j2n6s300_joint_end_effector
- removed joint j2n6s300_joint_finger_1
- removed joint j2n6s300_joint_finger_2
- removed joint j2n6s300_joint_finger_3
- removed joint j2n6s300_joint_finger_tip_1
- removed joint j2n6s300_joint_finger_tip_2
- removed joint j2n6s300_joint_finger_tip_3
- added joint m1n6s300_joint_1: type continuous, parent m1n6s300_link_base, child m1n6s300_link_1, origin xyz=0 0 0.15675 rpy=0 3.141592653589793 0, axis 0 0 1, limit effort=40 velocity=0.6283185307179586
- added joint m1n6s300_joint_2: type revolute, parent m1n6s300_link_1, child m1n6s300_link_2, origin xyz=0 0.0016 -0.11875 rpy=-1.5707963267948966 0 3.141592653589793, axis 0 0 1, limit lower=0.8726646259971648 upper=5.410520681182422 effort=80 velocity=0.6283185307179586
- added joint m1n6s300_joint_3: type revolute, parent m1n6s300_link_2, child m1n6s300_link_3, origin xyz=0 -0.290 0 rpy=0 3.141592653589793 0, axis 0 0 1, limit lower=0.6108652381980153 upper=5.672320068981571 effort=40 velocity=0.6283185307179586
- added joint m1n6s300_joint_4: type continuous, parent m1n6s300_link_3, child m1n6s300_link_4, origin xyz=0 0.1231 -0.0086 rpy=-1.5707963267948966 0 3.141592653589793, axis 0 0 1, limit effort=20 velocity=0.8377580409572781
- added joint m1n6s300_joint_5: type continuous, parent m1n6s300_link_4, child m1n6s300_link_5, origin xyz=0 -0.03703 -0.06414 rpy=1.0471975511965976 0 3.141592653589793, axis 0 0 1, limit effort=20 velocity=0.8377580409572781
- added joint m1n6s300_joint_6: type continuous, parent m1n6s300_link_5, child m1n6s300_link_6, origin xyz=0 -0.03703 -0.06414 rpy=1.0471975511965976 0 3.141592653589793, axis 0 0 1, limit effort=20 velocity=0.8377580409572781
- added joint m1n6s300_joint_base: type fixed, parent root, child m1n6s300_link_base, origin xyz=0 0 0 rpy=0 0 0, axis 0 0 0
- added joint m1n6s300_joint_end_effector: type fixed, parent m1n6s300_link_6, child m1n6s300_end_effector, origin xyz=0 0 -0.1600 rpy=3.141592653589793 0 1.5707963267948966, axis 0 0 0
- added joint m1n6s300_joint_finger_1: type revolute, parent m1n6s300_link_6, child m1n6s300_link_finger_1, origin xyz=0.00279 0.03126 -0.11467 rpy=-1.7047873384941834 0.6476144647144773 1.67317415161155, axis 0 0 1, limit lower=0 upper=1.51 effort=10 velocity=1
- added joint m1n6s300_joint_finger_2: type revolute, parent m1n6s300_link_6, child m1n6s300_link_finger_2, origin xyz=0.02226 -0.02707 -0.11482 rpy=-1.570796327 .649262481663582 -1.38614049188413, axis 0 0 1, limit lower=0 upper=1.51 effort=10 velocity=1
- added joint m1n6s300_joint_finger_3: type revolute, parent m1n6s300_link_6, child m1n6s300_link_finger_3, origin xyz=-0.02226 -0.02707 -0.11482 rpy=-1.570796327 .649262481663582 -1.75545216211587, axis 0 0 1, limit lower=0 upper=1.51 effort=10 velocity=1
- added joint m1n6s300_joint_finger_tip_1: type revolute, parent m1n6s300_link_finger_1, child m1n6s300_link_finger_tip_1, origin xyz=0.044 -0.003 0 rpy=0 0 0, axis 0 0 1, limit lower=0 upper=2 effort=10 velocity=1
- added joint m1n6s300_joint_finger_tip_2: type revolute, parent m1n6s300_link_finger_2, child m1n6s300_link_finger_tip_2, origin xyz=0.044 -0.003 0 rpy=0 0 0, axis 0 0 1, limit lower=0 upper=2 effort=10 velocity=1
- added joint m1n6s300_joint_finger_tip_3: type revolute, parent m1n6s300_link_finger_3, child m1n6s300_link_finger_tip_3, origin xyz=0.044 -0.003 0 rpy=0 0 0, axis 0 0 1, limit lower=0 upper=2 effort=10 velocity=1
- joint camera_joint: origin xyz=0.0 -0.7 0.5 rpy=0 0.785375 1.57075 -> xyz=0.4 0.4 0.5 rpy=0 0.785375 -1.57075; parent j2n6s300_link_base -> m1n6s300_link_base
