Commit message: Corregir posición de la cámara en el Kinova Mico

File: kinova_roscontrol/src/kinova-ros/kinova_description/urdf/m1n6s300.xacro (robot description, xacro)
@@ -110,5 +110,5 @@
         <!-- Camera parameters -->
         <xacro:camera_v0 parent="${prefix}_link_base">
-	     <origin xyz="0.4 0.4 0.5" rpy="0 0.785375 -1.57075"/>
+	     <origin xyz="0 0.4 0.5" rpy="0 0.785375 -1.57075"/>
         </xacro:camera_v0>
         <xacro:kinova_armlink link_name="${prefix}_link_1" link_mesh="${link_1_mesh}" use_ring_mesh="true" mesh_no="${link_1_mesh_no}"/>
