Commit message: Añadir cámara

File: kinova_roscontrol/src/kinova-ros/kinova_description/urdf/j2n6s300.xacro (robot description, xacro)
@@ -16,4 +16,6 @@
     <xacro:include filename="$(find kinova_description)/urdf/kinova_common.xacro" />
     <xacro:include filename="$(find kinova_description)/urdf/kinova_finger_set.xacro" />
+    <!-- Camera -->
+    <xacro:include filename="$(find kinova_description)/urdf/camera/camera.urdf.xacro"/>
     <!-- Import all Gazebo-customization elements -->
     <xacro:include filename="$(find kinova_description)/urdf/kinova.gazebo" />
@@ -98,4 +100,8 @@
         <xacro:kinova_armlink link_name="${prefix}_link_base" link_mesh="${link_base_mesh}" mesh_no="${link_base_mesh_no}"/>
         <xacro:kinova_armjoint joint_name="${prefix}_joint_base" type="${joint_base_type}" parent="${base_parent}" child="${prefix}_link_base" joint_axis_xyz="${joint_base_axis_xyz}" joint_origin_xyz="${joint_base_origin_xyz}" joint_origin_rpy="${joint_base_origin_rpy}" fixed="true"/>
+        <!-- Camera parameters -->
+        <xacro:camera_v0 parent="${prefix}_link_base">
+	     <origin xyz="0.0 -0.7 0.5" rpy="0 0.785375 1.57075"/>
+        </xacro:camera_v0>
         <xacro:kinova_armlink link_name="${prefix}_link_1" link_mesh="${link_1_mesh}" use_ring_mesh="true" mesh_no="${link_1_mesh_no}"/>
         <xacro:kinova_armjoint joint_name="${prefix}_joint_1" type="${joint_1_type}" parent="${prefix}_link_base" child="${prefix}_link_1" joint_axis_xyz="${joint_1_axis_xyz}" joint_origin_xyz="${joint_1_origin_xyz}" joint_origin_rpy="${joint_1_origin_rpy}" joint_velocity_limit="${joint_1_velocity_limit}" joint_torque_limit="${joint_1_torque_limit}"/>
@@ -114,3 +120,4 @@
     <xacro:kinova_3fingers link_hand="${prefix}_link_6" prefix="${prefix}_"/>
     </xacro:macro>
+    <xacro:camera_gazebo_v0 />
 </root>

File: kinova_roscontrol/src/kinova-ros/kinova_description/urdf/m1n6s300.xacro (robot description, xacro)
@@ -16,4 +16,6 @@
     <xacro:include filename="$(find kinova_description)/urdf/kinova_common.xacro" />
     <xacro:include filename="$(find kinova_description)/urdf/kinova_finger_set.xacro" />
+    <!-- Camera -->
+    <xacro:include filename="$(find kinova_description)/urdf/camera/camera.urdf.xacro"/>
     <!-- Import all Gazebo-customization elements -->
     <xacro:include filename="$(find kinova_description)/urdf/kinova.gazebo" />
@@ -106,4 +108,8 @@
         <xacro:kinova_armlink link_name="${prefix}_link_base" link_mesh="${link_base_mesh}" mesh_no="${link_base_mesh_no}"/>
         <xacro:kinova_armjoint joint_name="${prefix}_joint_base" type="${joint_base_type}" parent="${base_parent}" child="${prefix}_link_base" joint_axis_xyz="${joint_base_axis_xyz}" joint_origin_xyz="${joint_base_origin_xyz}" joint_origin_rpy="${joint_base_origin_rpy}" joint_lower_limit="0" joint_upper_limit="0" joint_velocity_limit="0" joint_torque_limit="0" fixed="true"/>
+        <!-- Camera parameters -->
+        <xacro:camera_v0 parent="${prefix}_link_base">
+	     <origin xyz="0.4 0.4 0.5" rpy="0 0.785375 -1.57075"/>
+        </xacro:camera_v0>
         <xacro:kinova_armlink link_name="${prefix}_link_1" link_mesh="${link_1_mesh}" use_ring_mesh="true" mesh_no="${link_1_mesh_no}"/>
         <xacro:kinova_armjoint joint_name="${prefix}_joint_1" type="${joint_1_type}" parent="${prefix}_link_base" child="${prefix}_link_1" joint_axis_xyz="${joint_1_axis_xyz}" joint_origin_xyz="${joint_1_origin_xyz}" joint_origin_rpy="${joint_1_origin_rpy}" joint_lower_limit="${joint_1_lower_limit}" joint_upper_limit="${joint_1_upper_limit}" joint_velocity_limit="${joint_1_velocity_limit}" joint_torque_limit="${joint_1_torque_limit}"/>
@@ -122,3 +128,4 @@
     <xacro:kinova_3fingers link_hand="${prefix}_link_6" prefix="${prefix}_"/>
     </xacro:macro>
+    <xacro:camera_gazebo_v0 />
 </root>

Commit message: Cambio posición cámara (completamente hacia abajo)

File: kinova_roscontrol/src/kinova-ros/kinova_description/urdf/j2n6s300.xacro (robot description, xacro)
@@ -102,5 +102,5 @@
         <!-- Camera parameters -->
         <xacro:camera_v0 parent="${prefix}_link_base">
-	     <origin xyz="0.0 -0.7 0.5" rpy="0 0.785375 1.57075"/>
+	     <origin xyz="0.0 -0.5 0.5" rpy="0 1.575375 1.57075"/>
         </xacro:camera_v0>
         <xacro:kinova_armlink link_name="${prefix}_link_1" link_mesh="${link_1_mesh}" use_ring_mesh="true" mesh_no="${link_1_mesh_no}"/>

Commit message: Cambio en la posición de la cámara

File: kinova_roscontrol/src/kinova-ros/kinova_description/urdf/j2n6s300.xacro (robot description, xacro)
@@ -102,5 +102,5 @@
         <!-- Camera parameters -->
         <xacro:camera_v0 parent="${prefix}_link_base">
-	     <origin xyz="0.0 -0.5 0.5" rpy="0 1.575375 1.57075"/>
+	     <origin xyz="0.0 -0.5 0.5" rpy="0 ${J_PI/2} ${J_PI/2}"/>
         </xacro:camera_v0>
         <xacro:kinova_armlink link_name="${prefix}_link_1" link_mesh="${link_1_mesh}" use_ring_mesh="true" mesh_no="${link_1_mesh_no}"/>

Commit message: Cambio en la posición de la cámara

File: kinova_roscontrol/src/kinova-ros/kinova_description/urdf/j2n6s300.xacro (robot description, xacro)
@@ -102,5 +102,5 @@
         <!-- Camera parameters -->
         <xacro:camera_v0 parent="${prefix}_link_base">
-	     <origin xyz="0.0 -0.5 0.5" rpy="0 ${J_PI/2} ${J_PI/2}"/>
+	     <origin xyz="0.0 -0.5 0.5" rpy="0 ${J_PI/2} ${-J_PI/2}"/>
         </xacro:camera_v0>
         <xacro:kinova_armlink link_name="${prefix}_link_1" link_mesh="${link_1_mesh}" use_ring_mesh="true" mesh_no="${link_1_mesh_no}"/>

Commit message: Añadir segunda camara al URDF

File: kinova_roscontrol/src/kinova-ros/kinova_description/urdf/j2n6s300.xacro (robot description, xacro)
@@ -18,4 +18,5 @@
     <!-- Camera -->
     <xacro:include filename="$(find kinova_description)/urdf/camera/camera.urdf.xacro"/>
+    <xacro:include filename="$(find kinova_description)/urdf/camera2/camera.urdf.xacro"/>
     <!-- Import all Gazebo-customization elements -->
     <xacro:include filename="$(find kinova_description)/urdf/kinova.gazebo" />
@@ -104,4 +105,7 @@
 	     <origin xyz="0.0 -0.5 0.5" rpy="0 ${J_PI/2} ${-J_PI/2}"/>
         </xacro:camera_v0>
+        <xacro:camera_v1 parent="${prefix}_link_base">
+	     <origin xyz="-0.35 0.35 0.5" rpy="0 ${J_PI/2} ${-J_PI/2}"/>
+        </xacro:camera_v1>
         <xacro:kinova_armlink link_name="${prefix}_link_1" link_mesh="${link_1_mesh}" use_ring_mesh="true" mesh_no="${link_1_mesh_no}"/>
         <xacro:kinova_armjoint joint_name="${prefix}_joint_1" type="${joint_1_type}" parent="${prefix}_link_base" child="${prefix}_link_1" joint_axis_xyz="${joint_1_axis_xyz}" joint_origin_xyz="${joint_1_origin_xyz}" joint_origin_rpy="${joint_1_origin_rpy}" joint_velocity_limit="${joint_1_velocity_limit}" joint_torque_limit="${joint_1_torque_limit}"/>
@@ -121,3 +125,4 @@
     </xacro:macro>
     <xacro:camera_gazebo_v0 />
+    <xacro:camera_gazebo_v1 />
 </root>
