Commit message: Elimina físicas de la cámara

File: kinova_roscontrol/src/kinova-ros/kinova_description/urdf/camera/camera.urdf.xacro (robot description, xacro)
@@ -14,14 +14,4 @@
 		</geometry>
 	  </visual>
-	  <collision>
-		<geometry>
-		  <mesh filename="package://kinova_description/meshes/STL/camera/camera.stl"/>
-		</geometry>
-	  </collision>
-	  <inertial>
-		<origin xyz="0 0 0"/>
-		<mass value="0.1"/>
-		<inertia ixx="0.00001" ixy="0" ixz="0" iyy="0.00001" iyz="0" izz="0.00001" />
-	  </inertial>
 	</link>
   </xacro:macro>
